File: pcb/arm_controller_board/arm_controller_board.kicad_sch (KiCad schematic)
At the start: 20 parts, among them J1 SERVO, J10 POT B1K, J11 POT B1K, J12 POT B1K, J2 LCD, J3 POT B1K, J4 PULSADOR, J5 CONSOLE, J6 PULSADOR, J7 PULSADOR, J8 POT B1K, J9 POT B1K

Commit message: feat(pcb): add HW-221 symbol and footprint and the first schematic
Parts:
- renumbered A2 to A1, A1 to A2, J2 to J1, J5 to J11, J1 to J12, J12 to J2, J11 to J3, J8 to J4, J3 to J5, J4 to J6, J6 to J7, J7 to J8
Other:
- note added: "Driver para servos STS3215 (Waveshare A): Conexión: 1 <-> TX 2 <-> RX 3 <-> GND Tiene su propia fuente de 12V. Solo se comparte GND. El jumper del driver tiene que ir en la posición A - UART. La alimentación del driver va a través de una parada de emergencia externa. No pasa por esta placa."
- note added: "HW-221: En el módulo, OE está conectado a VA."
- note added: "Pot gripper (joint 6) + navegación Conexión: 1 <-> 1 2 <-> 2 Medio 3 <-> 3"
- note removed: "Driver para servos ST3215 (Waveshare A): Conexión: 1 <-> TX 2 <-> RX 3 <-> GND Tiene su propia fuente de 12V. Solo se comparte GND. El jumper del driver tiene que ir en la posición A - UART."
- note removed: "HW-221: En el módulo, OE está conectado a VA;"
- note removed: "Pot gripper (joint 6) + navegación) Conexión: 1 <-> 1 2 <-> 2 Medio 3 <-> 3"

Commit message: docs(pcb): fill in the schematic title block
Other:
- company: (none) -> UTN FRBA - Proyecto Final
- title: (none) -> Placa controladora del brazo robótico
Changed lines of the file:
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@@
 	(generator_version "9.0")
 	(paper "A4")
+	(title_block
+		(title "Placa controladora del brazo robótico")
+		(date "2026-10-23")
+		(rev "1")
+		(company "UTN FRBA - Proyecto Final")
+		(comment 1 "Autor: Ezequiel Alegre Mendoza")
+	)
 	(text "Pot gripper (joint 6) + navegación\nConexión:\n1 <-> 1\n2 <-> 2 Medio\n3 <-> 3"
 		(exclude_from_sim no)
